File: EchoEarCopyProj.kicad_sch (KiCad schematic)
At the start: 7 parts, among them U1 ESP32-S3-WROOM-1-N32R16V

Commit message: before file cleaning 3.1.2026
Parts:
- removed C1: 10uF, C0603, symbol Device:C
- removed C2: 100nF, C0402, symbol Device:C
- removed C3: 10uF, C0402, symbol Device:C_Small
- removed R1, R2: 2.2k, R0402, symbol Device:R_Small
- removed R3: 10k, R0402, symbol Device:R_Small
- removed U1: ESP32-S3-WROOM-1-N32R16V, RF_Module:ESP32-S3-WROOM-1, symbol EchoEarCopy:ESP32-S3-WROOM-1-N32R16V
Connections:
- no-connect marks 3 -> 0
Other:
- added sheet Interface (Interface.kicad_sch)
- added sheet MCU (MCU.kicad_sch)
- note removed: "*"
- note removed: "BOOT"
- note removed: "CTRL"
- note removed: "I2C"
- note removed: "I2S"
- note removed: "INT"
- note removed: "LCD"
- note removed: "SD"
- note removed: "TOUCH"
- note removed: "UART1"
- note removed: "USB"
- title: (none) -> Overview
